Commit message: Added friction to prevent strange behaviour of one finger.

File: schunk_description/urdf/sdh/sdh.urdf.xacro (robot description, xacro)
@@ -54,5 +54,5 @@
 			<child link="${name}_finger_11_link"/>
 			<axis xyz="0 0 1" />
-			<dynamics damping="1" />
+			<dynamics damping="10.0" friction="20000.0" />
 			<limit effort="100" lower="0" upper="1.570796327" velocity="5"/>
 		</joint>
@@ -143,5 +143,5 @@
 			<child link="${name}_finger_21_link"/>
 			<axis xyz="0 0 -1" />
-			<dynamics damping="1" />
+			<dynamics damping="10.0" friction="20000.0" />
 			<limit effort="100" lower="0" upper="1.570796327" velocity="5"/>
 		</joint>
@@ -230,4 +230,5 @@
 			<parent link="${name}_palm_link"/>
 			<child link="${name}_thumb_1_link"/>
+			<dynamics damping="10.0" friction="20000.0" />
 		</joint>
 		<link name="${name}_thumb_1_link">
